File: Sthymuli-cardinalboard.kicad_pro.kicad_pcb (KiCad board)
At the start: 2 copper layers, 153.6 x 35.9 mm, 30 parts, among them J1 Conn_02x08_Counter_Clockwise, Q1 NX7002AK, Q2 NX7002AK, SW1 SW_Push, SW2 SW_Push, U1 ITR9909, U2 ITR9909, U3 LSM6DS3

Commit message: regenerated output
Parts:
- removed the REF** at (97.8, 100.8)
- added REF**: OSHW-Logo_19x20mm_SilkScreen, Symbol:OSHW-Logo_19x20mm_SilkScreen, F.Cu at (173.7, 92.6)
Connections:
- net btn_DOWN renamed btn_A
- net btn_UP renamed btn_B

Commit message: fixed resistor footprint, enabled all DRC, improved readability
Parts:
- removed D2: D_Schottky, Diode_SMD:D_SOD-123F
- removed F1: Fuse, Resistor_SMD:R_0805_2012Metric
- added Q3: Q_PMOS_GSD, Package_TO_SOT_SMD:TSOT-23, F.Cu at (109.9, 89.5)
- added R5: 100K, Resistor_SMD:R_0603_1608Metric, F.Cu at (167.1, 84.3)
- added R6: 100K, Resistor_SMD:R_0603_1608Metric, F.Cu at (167.1, 78.2)
- R1, R2, R3, R4: footprint Capacitor_SMD:C_0201_0603Metric -> Resistor_SMD:R_0603_1608Metric
- moved REF** 2.06 mm to (175.6, 93.2)
- moved Q1 1.30 mm to (167.0, 75.2)
- moved R1 0.89 mm to (144.9, 79.4)
- moved C3 0.35 mm to (144.8, 73.2)
- moved R4 0.22 mm to (159.1, 74.6)
- moved R3 0.18 mm to (156.6, 78.5)
Routing:
- net BAT-: track 124.6 -> 136.5 mm, vias 2 -> 3
- net GND: track 245.1 -> 248.9 mm
- net Net-(BT1-+): track 4.87 -> 7.89 mm, vias 1 -> 2
- net BAT+: track 14.3 -> 11.6 mm, vias 1 -> 2
- net Net-(Q1-D): track 19.2 -> 17.1 mm, vias 0 -> 2
- net IR_TRA_HORI: track 105.7 -> 107.2 mm
- net +3V3: track 117.3 -> 118.6 mm
- net IR_REC_HORI: track 73.9 -> 74.7 mm
- net Net-(D5-DOUT): track 50.3 -> 50.9 mm
- net Net-(R3-Pad1): track 6.45 -> 5.87 mm
Other:
- board text added: "Sthymuli cardinalboard v1.1 (2026) Nathann Morand Manuel BL"
- board text removed: "Sthymuli cardinalboard v1.0 (2026) Nathann Morand Manuel BL"
